File: Inteligent_Robot/Main_Bord.sch (EAGLE design)
At the start: 77 parts, among them CN5 DF11-4DS-2C, CN6 DF11-4DS-2C, CN7 IL-G_ST_4, CN8 IL-G_ST_4, IC1 TWE-001L-IP, IC2 LTC2862A, IC3 A4988, IC4 A4988

Commit message: Start Print section
Parts:
- removed C10, C11, C12, C13, C14, C15, C16, C17, C18, C9: GMR31, Murata:GMR31
- removed DC13, DC14: YFF21PC, TDK:YFF21PC
- removed IC3, IC4: A4988, Allegro:A4988
- removed OS-CON1, OS-CON2: 16SVPS100M, OS-CON:16SVPS100M
- removed RA5, RA6: EXB-38V103JV, Pana_Chip_RA:EXB-38V103JV
- removed U$19, U$20, U$21, U$22, U$29, U$30, U$31, U$32, U$33, U$35: MCR03, ROHM:MCR03
- removed VR1, VR2: G43ATB103, tocos:G43ATB103
- added C22, C23, C24, C25, C26, C27, C34, C35, C36, C37, C38, C39: 0.1μ, Murata:GRM033R61C104KE14
- added DC15, DC17: YFF21PC, TDK:YFF21PC
- added IC5, IC7: A4988, Allegro:A4988
- added OS-CON3, OS-CON5: 16SVPS100M, OS-CON:16SVPS100M
- added R13, R14, R15, R16, R3, R4, R7, R8: MCR006, ROHM:MCR006
- added RA12, RA13, RA8, RA9: EXB-38V103JV, Pana_Chip_RA:EXB-38V103JV
- added RS3, RS4, RS7, RS8: LTR10EVHFLR110, ROHM:LTR10EVHFLR110
- added VR3, VR5: G43ATB103, tocos:G43ATB103
Connections:
- removed net DIR3: IC3.SENSE1, U$30.1
- removed net DIR4: IC4.SENSE1, U$32.1
- removed net N$10: U$21.1, VR1.2
- removed net N$11: U$22.1, VR2.2
- removed net N$12: IC4.VREF, VR2.IO3
- removed net N$16: IC4.MS3, RA6-3.1
- removed net N$17: IC3.SENSE2, U$29.1
- removed net N$18: IC4.SENSE2, U$31.1
- removed net N$19: C12.2, IC3.VCP
- removed net N$20: C16.2, IC4.VCP
- removed net N$21: C11.2, IC3.CP1
- removed net N$22: C11.1, IC3.CP2
- removed net N$23: C15.2, IC4.CP1
- removed net N$24: C15.1, IC4.CP2
- removed net N$25: IC4.ENABLE, RA6-4.1
- removed net N$26: C10.1, IC3.VREG
- removed net N$27: IC3.ROSC, U$33.2
- removed net N$28: C14.1, IC4.VREG
- removed net N$29: IC4.ROSC, U$35.2
- removed net N$30: IC3.RESET, U$19.1
- removed net N$31: IC4.RESET, U$20.1
- removed net N$32: IC4.MS2, RA6-2.1
- removed net N$33: IC4.MS1, RA6-1.1
- removed net N$34: IC3.MS3, RA5-3.1
- removed net N$35: IC3.MS2, RA5-2.1
- removed net N$42: IC3.MS1, RA5-1.1
- removed net N$45: C9.1, DC13.P$1, IC3.VDD, VR1.1
- removed net N$46: C13.1, DC14.P$1, IC4.VDD, VR2.1
- removed net N$6: IC3.ENABLE, RA5-4.1
- removed net N$9: IC3.VREF, VR1.IO3
- new net +3.3V: C1.1, C2.1, DC10.P$1, DC12.P$2, DC5.P$2, RA4-1.2, RA4-2.2, RA4-3.2, RA4-4.2
- new net +5V: C19.1, C20.1, C5.1, C8.1, CN2.1, CN3.1, CN4.1, DC8.P$1, U$12.1, U$13.1, U$14.1, U$15.1
- new net DIR: IC5.DIR, IC7.DIR, R15.1, R7.1
- new net DIR5: IC5.SENSE1, RS3.1
- new net DIR7: IC7.SENSE1, RS7.1
- new net MS1: IC5.MS1, IC7.MS1, RA12-1.1, RA8-1.1
- new net MS2: IC5.MS2, IC7.MS2, RA12-2.1, RA8-2.1
- new net MS3: IC5.MS3, IC7.MS3, RA12-3.1, RA8-3.1
- new net MT_1A: IC5.OUT1A
- new net MT_1B: IC5.OUT1B
- new net MT_2A: IC5.OUT2A
- new net MT_2B: IC5.OUT2B
- new net N$101: C35.1, IC7.VCP
- new net N$102: C36.1, IC7.CP1
- new net N$103: C36.2, IC7.CP2
- new net N$104: IC7.SENSE2, RS8.1
- new net N$105: C37.2, IC7.VREG
- new net N$106: IC7.ROSC, RA13-3.1
- new net N$107: IC7.ENABLE, R16.1
- new net N$108: IC7.RESET, RA13-2.1
- new net N$109: R13.2, VR5.2
- new net N$110: IC7.VREF, VR5.IO3
- new net N$111: DC17.P$1, IC7.VDD
- new net N$47: DC11.P$1
- new net N$57: C23.1, IC5.VCP
- new net N$58: C24.1, IC5.CP1
- new net N$59: C24.2, IC5.CP2
- new net N$60: IC5.SENSE2, RS4.1
- new net N$61: C25.2, IC5.VREG
- new net N$62: IC5.ROSC, RA9-3.1
- new net N$63: IC5.ENABLE, R8.1
- new net N$64: IC5.RESET, RA9-2.1
- new net N$65: R3.2, VR3.2
- new net N$66: IC5.VREF, VR3.IO3
- new net N$67: DC15.P$1, IC5.VDD
- new net STP: IC5.STEP, IC7.STEP, R14.1, R4.1
- new net VDD: C22.1, C23.2, C27.1, C34.1, C35.2, C39.1, C6.1, C7.1, CN1.1, CN5.3, CN6.3, DC-DC3.+VIN@1, DC-DC3.+VIN@2, DC-DC4.+VIN@1, DC-DC4.+VIN@2, IC5.VBB1, IC5.VBB2, IC7.VBB1, IC7.VBB2, OS-CON3.+, OS-CON5.+, U$9.+, XT60-1.1+
- net DIR1: no longer IC3.DIR
- net DIR2: no longer IC4.DIR
- net GND: now also C22.2, C25.1, C26.2, C27.2, C34.2, C37.1, C38.2, C39.2, DC15.GND, DC17.GND, IC5.GND, IC5.N.C., IC5.PAD, IC7.GND, IC7.N.C., IC7.PAD, OS-CON3.2, OS-CON5.2, R13.1, R14.2, R15.2, R16.2, R3.1, R4.2, R7.2, R8.2, RA12-1.2, RA12-2.2, RA12-3.2, RA13-2.2, RA13-3.2, RA13-4.2, RA8-1.2, RA8-2.2, RA8-3.2, RA9-2.2, RA9-3.2, RA9-4.2, RS3.2, RS4.2, RS7.2, RS8.2; no longer C10.2, C13.2, C14.2, C17.2, C18.2, C9.2, DC13.GND, DC14.GND, IC3.GND, IC3.N.C., IC3.PAD, IC4.GND, IC4.N.C., IC4.PAD, OS-CON1.2, OS-CON2.2, RA5-1.2, RA5-2.2, RA5-3.2, RA5-4.2, RA6-1.2, RA6-2.2, RA6-3.2, RA6-4.2, U$19.2, U$20.2, U$21.2, U$22.2, U$29.2, U$30.2, U$31.2, U$32.2, U$33.1, U$35.1
- net MT1_1A: no longer IC3.OUT1A
- net MT1_1B: no longer IC3.OUT1B
- net MT1_2A: no longer IC3.OUT2A
- net MT1_2B: no longer IC3.OUT2B
- net MT2_1A: now also IC7.OUT1A; no longer IC4.OUT1A
- net MT2_1B: now also IC7.OUT1B; no longer IC4.OUT1B
- net MT2_2A: now also IC7.OUT2A; no longer IC4.OUT2A
- net MT2_2B: now also IC7.OUT2B; no longer IC4.OUT2B
- net SLEEP1: now also IC5.SLEEP, IC7.SLEEP, RA13-4.1, RA9-4.1; no longer IC3.SLEEP, IC4.SLEEP
- net STP1: no longer IC3.STEP
- net STP2: no longer IC4.STEP
- net VCC: now also C26.1, C38.1, DC15.P$2, DC17.P$2, VR3.1, VR5.1; no longer C1.1, C12.1, C16.1, C17.1, C18.1, C19.1, C2.1, C20.1, C5.1, C6.1, C7.1, C8.1, CN1.1, CN2.1, CN3.1, CN4.1, CN5.3, CN6.3, DC-DC3.+VIN@1, DC-DC3.+VIN@2, DC-DC4.+VIN@1, DC-DC4.+VIN@2, DC10.P$1, DC11.P$1, DC12.P$2, DC13.P$2, DC14.P$2, DC5.P$2, DC8.P$1, IC3.VBB1, IC3.VBB2, IC4.VBB1, IC4.VBB2, OS-CON1.+, OS-CON2.+, RA4-1.2, RA4-2.2, RA4-3.2, RA4-4.2, U$12.1, U$13.1, U$14.1, U$15.1, U$9.+, XT60-1.1+

Commit message: Complete_First_version
Parts:
- removed U$18: MCR03, ROHM:MCR03
- added R1: MCR006, ROHM:MCR006
Connections:
- removed net DIR: IC5.DIR, IC7.DIR, R15.1, R7.1
- removed net MT_1A: IC5.OUT1A
- removed net MT_1B: IC5.OUT1B
- removed net MT_2A: IC5.OUT2A
- removed net MT_2B: IC5.OUT2B
- removed net N$47: DC11.P$1
- removed net STP: IC5.STEP, IC7.STEP, R14.1, R4.1
- removed net VCC: C26.1, C38.1, DC15.P$2, DC17.P$2, VR3.1, VR5.1
- net +5V: now also C26.1, C38.1, DC11.P$1, DC15.P$2, DC17.P$2, VR3.1, VR5.1
- net A*: now also DC3.P$1; no longer DC3.P$2
- net DIR1: now also IC5.DIR, R7.1; no longer RA1-2.1
- net DIR2: now also IC7.DIR, R15.1; no longer RA1-1.1
- net GND: no longer RA1-1.2, RA1-2.2, RA2-1.2, RA2-2.2, RA3-3.2
- net MT1_1A: now also CN7.3, IC5.OUT1A; no longer CN7.4
- net MT1_1B: now also CN7.4, IC5.OUT1B; no longer CN7.3
- net MT1_2A: now also IC5.OUT2A
- net MT1_2B: now also IC5.OUT2B
- net MT2_1A: now also CN8.3; no longer CN8.4
- net MT2_1B: now also CN8.4; no longer CN8.3
- net N$14: now also DC3.P$2, R1.1; no longer DC3.P$1, U$18.2
- net N$15: now also R1.2; no longer U$18.1
- net SLEEP1: no longer RA3-3.1
- net STP1: now also IC5.STEP, R4.1; no longer RA2-1.1
- net STP2: now also IC7.STEP, R14.1; no longer RA2-2.1
Other:
- moved on the sheet: DC3
